File: hardware/ctm_battery_adapter.kicad_pcb (KiCad board)
At the start: 2 copper layers, 50 x 10 mm, 29 parts, among them J1 USB_B_Micro, J2 Conn_01x02, J3 Conn_01x02, SW1 SW_Push_SPST_Shielded, U1 IP5306_CK, U2 AP63203WU, U3 RT9080-30GJ5

Commit message: Add files via upload
Parts:
- removed C9: 100n, Capacitor_SMD:C_0402_1005Metric
- removed REF**: enclosure, slk:enclosure
- C6: value 10u -> 4.7u
- C7: value 22u -> 10u
- D1, D2, D3, D4: footprint slk:LED_0402 -> slk:LED_RA_0402
- U2: value AP63203WU -> RT8010; footprint Package_TO_SOT_SMD:TSOT-23-6 -> slk:WDFN-6L_2x2
- U3: value RT9080-30GJ5 -> TLV75730PDRV; footprint Package_TO_SOT_SMD:TSOT-23-5 -> slk:WSON-6_2x2
- moved U3 2.48 mm to (90.4, 70.4), turned to 90 degrees
- moved L2 1.86 mm to (90.5, 67.7)
- moved C8 1.37 mm to (90.4, 72.4), turned to 0 degrees
- moved C7 1.13 mm to (93.1, 69.5)
- moved C6 1.00 mm to (95.4, 67.8)
- moved U2 0.44 mm to (93.1, 67.6)
- moved C3 0.16 mm to (98.5, 68.6)
- turned R4 to -90 degrees
- renumbered R3 to R1, R4 to R2, R1 to R3, R2 to R4
Connections:
- L2 pad 1: Net-(U2-SW) -> Net-(U2-LX)
- U2 pad 1: +3V3 -> unconnected-(U2-IC-Pad1)
- U2 pad 4: GND -> Net-(U2-LX)
- U2 pad 5: Net-(U2-SW) -> GND
- U2 pad 6: Net-(U2-BST) -> +3V3
- U3 pad 1: +3V3 -> +3V0
- U3 pad 2: GND -> unconnected-(U3-NC-Pad2)
- U3 pad 3: +3V3 -> GND
- U3 pad 4: unconnected-(U3-NC-Pad4) -> +3V3
- U3 pad 5: +3V0 -> unconnected-(U3-NC-Pad5)
Routing:
- net GND: track 15.5 -> 8.97 mm, vias 79 -> 84
- net +3V0: track 1.12 -> 6.28 mm
- net +3V3: track 3.32 -> 5.78 mm
- net Net-(U2-LX): track 0.00 -> 2.35 mm
- net +5V: track 7.46 -> 5.44 mm
- net VBUS: track 4.73 -> 6.54 mm
- net Net-(D1-A): track 1.77 -> 3.52 mm
- net Net-(U1-LED2): track 27.4 -> 29.0 mm
- net Net-(D3-A): track 2.24 -> 3.54 mm
- net Net-(U2-BST): track 1.23 -> 0.00 mm
- removed copper zone on F.Cu, net +3V0
- removed copper zone on F.Cu, net +3V3
- removed copper zone on F.Cu, net Net-(U2-SW)
Other:
- board text added: "CTM Battery Adapter Version 1.0.0 3/8/23"
- board text removed: "CTM Battery Adapter v1.0.0c 3/14/23"
