File: hardware/ctm_battery_adapter.kicad_sch (KiCad schematic)
At the start: 28 parts, among them J1 USB_B_Micro, J2 Conn_01x02, J3 Conn_01x02, SW1 SW_Push_SPST_Shielded, U1 IP5306_CK, U2 AP63203WU, U3 RT9080-30GJ5

Commit message: Add files via upload
Parts:
- removed C9: 100n, Capacitor_SMD:C_0402_1005Metric, symbol Device:C
- removed U2: AP63203WU, Package_TO_SOT_SMD:TSOT-23-6, symbol Regulator_Switching:AP63203WU
- removed U3: RT9080-30GJ5, Package_TO_SOT_SMD:TSOT-23-5, symbol slk:RT9080-30GJ5_TSOT-23-5
- added U2: RT8010, slk:WDFN-6L_2x2, symbol slk:RT8010
- added U3: TLV75730PDRV, slk:WSON-6_2x2, symbol Regulator_Linear:TLV75730PDRV
- C6: value 10u -> 4.7u
- C7: value 22u -> 10u
- D1, D2, D3, D4: footprint slk:LED_0402 -> slk:LED_RA_0402
- renumbered R3 to R1, R4 to R2, R1 to R3, R2 to R4
Connections:
- net +3V0: now also U3.1 (OUT)
- net +3V3: now also U2.6 (VOUT), U3.4 (EN), U3.6 (IN)
- net +5V: now also U2.2 (EN), U2.3 (VIN)
- net GND: now also U2.5 (GND), U2.7 (EPAD), U3.3 (GND), U3.7 (GND)
- net at L2.1: now also U2.4 (LX)
Other:
- moved on the sheet: L2
